File: hardware/pcb/Generator_hat/Generator_hat.kicad_pcb (KiCad board)
At the start: 2 copper layers, 69.1 x 53.8 mm, 18 parts, among them J1 Screw_Terminal_01x03, J2 Screw_Terminal_01x02, U1 DHT11

Commit message: updated ppt
Changed lines of the file:
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@@
   (segment (start 135.89 79.756) (end 125.73 79.756) (width 2) (layer "B.Cu") (net 13))
   (segment (start 103.632 67.056) (end 103.632 97.79) (width 0.254) (layer "F.Cu") (net 20))
+  (segment (start 132.32 61) (end 130.582 62.738) (width 0.254) (layer "F.Cu") (net 20))
+  (segment (start 130.582 62.738) (end 107.95 62.738) (width 0.254) (layer "F.Cu") (net 20))
   (segment (start 107.95 62.738) (end 103.632 67.056) (width 0.254) (layer "F.Cu") (net 20))
-  (segment (start 131.447237 61) (end 129.709237 62.738) (width 0.254) (layer "F.Cu") (net 20))
-  (segment (start 129.709237 62.738) (end 107.95 62.738) (width 0.254) (layer "F.Cu") (net 20))
   (segment (start 103.632 97.79) (end 108.712 97.79) (width 0.254) (layer "F.Cu") (net 20))
-  (segment (start 132.32 61) (end 131.447237 61) (width 0.254) (layer "F.Cu") (net 20))
   (segment (start 108.712 97.79) (end 109.982 96.52) (width 0.254) (layer "F.Cu") (net 20))
   (segment (start 107.188 100.33) (end 109.982 103.124) (width 0.25) (layer "F.Cu") (net 21))

Commit message: update pcb
Parts:
- added C3: 100nF, Capacitor_SMD:C_0805_2012Metric_Pad1.18x1.45mm_HandSolder, F.Cu at (140.0, 97.3)
- added C4: 22uF, Capacitor_SMD:CP_Elec_8x6.9, F.Cu at (124.7, 94.7)
- added C5: 100nF, Capacitor_SMD:C_0805_2012Metric_Pad1.18x1.45mm_HandSolder, F.Cu at (108.2, 95.0)
- added C6: 100nF, Capacitor_SMD:C_0805_2012Metric_Pad1.18x1.45mm_HandSolder, F.Cu at (148.3, 63.8)
- added C7: 100nF, Capacitor_SMD:C_0805_2012Metric_Pad1.18x1.45mm_HandSolder, F.Cu at (156.0, 63.8)
- added Chf1: 220nF, Capacitor_SMD:C_0805_2012Metric_Pad1.18x1.45mm_HandSolder, F.Cu at (126.5, 101.3)
- added Cin1: 4.7nF, Capacitor_SMD:C_0805_2012Metric_Pad1.18x1.45mm_HandSolder, F.Cu at (124.2, 101.3)
- added Cvcc1: 1uF, Capacitor_SMD:C_0805_2012Metric_Pad1.18x1.45mm_HandSolder, F.Cu at (142.0, 102.1)
- added L1: 2.2uH, Inductor_SMD:L_Taiyo-Yuden_NR-50xx_HandSoldering, F.Cu at (134.6, 93.2)
- added R6: 100k, Resistor_SMD:R_0805_2012Metric_Pad1.20x1.40mm_HandSolder, F.Cu at (134.6, 104.4)
- added R7: 100k, Resistor_SMD:R_0805_2012Metric_Pad1.20x1.40mm_HandSolder, F.Cu at (143.3, 97.3)
- added R8: 24.9k, Resistor_SMD:R_0805_2012Metric_Pad1.20x1.40mm_HandSolder, F.Cu at (140.0, 102.1)
- added R9: 10K, Resistor_SMD:R_0805_2012Metric_Pad1.20x1.40mm_HandSolder, F.Cu at (152.9, 64.5)
- added U2: LMR33610BDDAR, Package_SO:Texas_HSOP-8-1EP_3.9x4.9mm_P1.27mm_ThermalVias, F.Cu at (134.6, 99.1)
- D1, D2, D3, D4, D5, D6: footprint Diode_THT:D_DO-41_SOD81_P10.16mm_Horizontal -> Diode_SMD:D_SMA
- R2, R3, R4, R5: footprint Resistor_THT:R_Axial_DIN0207_L6.3mm_D2.5mm_P10.16mm_Horizontal -> Resistor_SMD:R_0805_2012Metric_Pad1.20x1.40mm_HandSolder
- moved R4 22.3 mm to (124.7, 73.7)
- moved R3 13.2 mm to (124.7, 75.7)
- moved R5 12.7 mm to (100.8, 69.1)
- moved C2 7.60 mm to (117.1, 68.3), turned to 180 degrees
- moved C1 7.58 mm to (117.1, 85.1), turned to 180 degrees
- moved D2 6.75 mm to (128.5, 68.3)
- moved D4 6.75 mm to (138.7, 68.3)
- moved D6 6.67 mm to (148.8, 68.3)
- moved R2 2.91 mm to (108.2, 98.8)
- moved D3 2.90 mm to (138.7, 80.5)
- moved D1 2.90 mm to (128.5, 80.5)
- moved D5 2.90 mm to (148.8, 80.5)
- moved R1 1.85 mm to (140.2, 87.1)
- moved J2 1.64 mm to (158.9, 87.1)
Connections:
- A1 pad 10: LOAD-GND -> Net-(A1-Pad10)
- A1 pad 5: unconnected-(A1-Pad5) -> +5V
- A1 pad 8: V-GEN -> unconnected-(A1-Pad8)
- C1 pad 1: V-GEN -> VDC
- C2 pad 1: V-GEN -> VDC
- D1 pad 1: V-GEN -> VDC
- D3 pad 1: V-GEN -> VDC
- D5 pad 1: V-GEN -> VDC
- J2 pad 2: V-GEN -> VDC
- R2 pad 1: +3V3 -> +5V
- R3 pad 1: V-GEN -> VDC
- U1 pad 1: +3V3 -> +5V
Routing:
- net VDC: track 0.00 -> 258.1 mm, vias 0 -> 5
- net V-GEN: track 112.3 -> 0.00 mm
- net +5V: track 0.00 -> 88.6 mm, vias 0 -> 3
- net +3V3: track 68.8 -> 0.00 mm
- net V-SENSE: track 90.6 -> 36.6 mm, vias 0 -> 1
- net LOAD-GND: track 48.5 -> 33.6 mm
- net Net-(Cvcc1-Pad1): track 0.00 -> 13.0 mm
- net LED: track 50.4 -> 61.8 mm, vias 0 -> 1
- net Net-(D5-Pad2): track 17.7 -> 26.0 mm, vias 0 -> 1
- net Net-(R7-Pad2): track 0.00 -> 7.89 mm, vias 0 -> 2
- net Net-(C3-Pad1): track 0.00 -> 6.79 mm
- net Net-(A1-Pad10): track 0.00 -> 5.87 mm
- net Net-(R6-Pad1): track 0.00 -> 4.13 mm
- net Net-(D7-Pad2): track 6.10 -> 2.55 mm
- net GND: track 0.00 -> 3.36 mm, vias 0 -> 14
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